File: jlcpcb_2_layer/jlcpcb_2_layer.sch (KiCad schematic (older format))
At the start: 2 parts

Commit message: updated JLCPCB 2layer template with new date
Parts:
- N2: value V20171120 -> V20180719
Changed lines of the file:
@@
 LIBS:SquantorPCBOutline
 LIBS:SquantorProto
+LIBS:jlcpcb_2_layer-cache
 EELAYER 25 0
 EELAYER END
@@
 P 850 7700
 F 0 "N2" H 850 7800 60  0000 C CNN
-F 1 "V20171120" H 850 7700 60  0000 C CNN
+F 1 "V20180719" H 850 7700 60  0000 C CNN
 F 2 "SquantorLabels:Label_version" H 850 7700 60  0001 C CNN
 F 3 "" H 850 7700 60  0001 C CNN

Commit message: updated JLCPCB 2layer template to kicad 5
Parts:
- N1: symbol OHWLOGO -> SquantorLabels:OHWLOGO
- N2: value V20180719 -> V20180826; symbol VYYYYMMDD -> SquantorLabels:VYYYYMMDD
Changed lines of the file:
@@
-EESchema Schematic File Version 2
-LIBS:power
-LIBS:device
-LIBS:switches
-LIBS:relays
-LIBS:motors
-LIBS:transistors
-LIBS:conn
-LIBS:linear
-LIBS:regul
-LIBS:74xx
-LIBS:cmos4000
-LIBS:adc-dac
-LIBS:memory
-LIBS:xilinx
-LIBS:microcontrollers
-LIBS:dsp
-LIBS:microchip
-LIBS:analog_switches
-LIBS:motorola
-LIBS:texas
-LIBS:intel
-LIBS:audio
-LIBS:interface
-LIBS:digital-audio
-LIBS:philips
-LIBS:display
-LIBS:cypress
-LIBS:siliconi
-LIBS:opto
-LIBS:atmel
-LIBS:contrib
-LIBS:valves
-LIBS:SquantorButtons
-LIBS:SquantorConnectors
-LIBS:SquantorLabels
-LIBS:SquantorPCBOutline
-LIBS:SquantorProto
+EESchema Schematic File Version 4
 LIBS:jlcpcb_2_layer-cache
-EELAYER 25 0
+EELAYER 26 0
 EELAYER END
 $Descr A4 11693 8268
@@
 $EndDescr
 $Comp
-L VYYYYMMDD N2
+L SquantorLabels:VYYYYMMDD N2
 U 1 1 5A1357A5
 P 850 7700
 F 0 "N2" H 850 7800 60  0000 C CNN
-F 1 "V20180719" H 850 7700 60  0000 C CNN
+F 1 "V20180826" H 850 7700 60  0000 C CNN
 F 2 "SquantorLabels:Label_version" H 850 7700 60  0001 C CNN
 F 3 "" H 850 7700 60  0001 C CNN
@@
 $EndComp
 $Comp
-L OHWLOGO N1
+L SquantorLabels:OHWLOGO N1
 U 1 1 5A135869
 P 850 7350
