File: Hammond_1593K_OSH2layer/Hammond_1593K_OSH2layer.kicad_pcb (KiCad board)
At the start: 2 copper layers, 2 parts

Commit message: updated Hammond 1593 OSHPark 2 layer template
Parts:
- N2: value V20171120 -> V20180726
Changed lines of the file:
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@@
-(kicad_pcb (version 4) (host pcbnew 4.0.7-e2-6376~58~ubuntu17.04.1)
+(kicad_pcb (version 20171130) (host pcbnew 5.0.0-fee4fd1~65~ubuntu18.04.1)
   (general
-    (links 0)
-    (no_connects 0)
-    (area 0 0 0 0)
     (thickness 1.6)
     (drawings 0)
@@
       (layerselection 0x00030_80000001)
       (usegerberextensions false)
+      (usegerberattributes false)
+      (usegerberadvancedattributes false)
+      (creategerberjobfile false)
       (excludeedgelayer true)
       (linewidth 0.100000)
@@
       (hpglpennumber 1)
       (hpglpenspeed 20)
-      (hpglpendiameter 15)
-      (hpglpenoverlay 2)
+      (hpglpendiameter 15.000000)
       (psnegative false)
       (psa4output false)
@@
       (effects (font (size 1 1) (thickness 0.15)))
     )
-    (fp_text value V20171120 (at 0 0) (layer F.SilkS)
-      (effects (font (size 1 1) (thickness 0.15)))
-    )
+    (fp_text value V20180726 (at 0 0) (layer F.SilkS)
+      (effects (font (size 1 1) (thickness 0.15)))
+    )
