File: NiBeetle_JLCPCB_4layer/NiBeetle_JLCPCB_4layer.sch (KiCad schematic (older format))
At the start: 2 parts

Commit message: updated Nickel beetle template project
Parts:
- added J1: DevBoardDigital, SquantorConnectors:Header-0127-2X10-H006, symbol SquantorConnectors:DevBoardDigital
- added J2: DevBoardAnalog, SquantorConnectors:Header-0127-2X10-H006, symbol SquantorConnectors:DevBoardAnalog
- added MH1, MH2: MountingHole, SquantorPcbOutline:MountingHole_2.5mm_no_metal, symbol Mechanical:MountingHole
Connections:
- net labels added: VCC, VDD, VDDA, VSS, VSSA
- wire segments 0 -> 12
Changed lines of the file:
@@
+	1    0    0    -1
+$EndComp
+$Comp
+L power:VDD #PWR0101
+U 1 1 5B7AAAB8
+P 2150 1000
+F 0 "#PWR0101" H 2150 850 50  0001 C CNN
+F 1 "VDD" V 2167 1128 50  0000 L CNN
+F 2 "" H 2150 1000 50  0001 C CNN
+F 3 "" H 2150 1000 50  0001 C CNN
+	1    2150 1000
+	0    1    1    0
+$EndComp
+$Comp
+L power:VSS #PWR0102
+U 1 1 5B7AAB25
+P 2150 1100
+F 0 "#PWR0102" H 2150 950 50  0001 C CNN
+F 1 "VSS" V 2167 1228 50  0000 L CNN
+F 2 "" H 2150 1100 50  0001 C CNN
+F 3 "" H 2150 1100 50  0001 C CNN
+	1    2150 1100
+	0    1    1    0
+$EndComp
+$Comp
+L power:VDD #PWR0103
+U 1 1 5B7AAB40
+P 950 1000
+F 0 "#PWR0103" H 950 850 50  0001 C CNN
+F 1 "VDD" V 968 1127 50  0000 L CNN
+F 2 "" H 950 1000 50  0001 C CNN
+F 3 "" H 950 1000 50  0001 C CNN
+	1    950  1000
+	0    -1   -1   0
+$EndComp
+$Comp
+L power:VSS #PWR0104
+U 1 1 5B7AAB57
+P 950 1100
+F 0 "#PWR0104" H 950 950 50  0001 C CNN
+F 1 "VSS" V 968 1228 50  0000 L CNN
+F 2 "" H 950 1100 50  0001 C CNN
+F 3 "" H 950 1100 50  0001 C CNN
+	1    950  1100
+	0    -1   -1   0
+$EndComp
+Wire Wire Line
+	950  1000 1000 1000
+Wire Wire Line
+	1000 1100 950  1100
+Wire Wire Line
+	2100 1000 2150 1000
+Wire Wire Line
+	2150 1100 2100 1100
+$Comp
+L SquantorConnectors:DevBoardDigital J1
+U 1 1 5B7AC4CB
+P 1550 1450
+F 0 "J1" H 1550 2187 60  0000 C CNN
+F 1 "DevBoardDigital" H 1550 2081 60  0000 C CNN
+F 2 "SquantorConnectors:Header-0127-2X10-H006" H 1550 1850 60  0001 C CNN
+F 3 "" H 1550 1850 60  0001 C CNN
+	1    1550 1450
+	1    0    0    -1
+$EndComp
+$Comp
+L SquantorConnectors:DevBoardAnalog J2
+U 1 1 5B7AC569
+P 1550 2800
+F 0 "J2" H 1550 3537 60  0000 C CNN
+F 1 "DevBoardAnalog" H 1550 3431 60  0000 C CNN
+F 2 "SquantorConnectors:Header-0127-2X10-H006" H 1550 3200 60  0001 C CNN
+F 3 "" H 1550 3200 60  0001 C CNN
+	1    1550 2800
+	1    0    0    -1
+$EndComp
+$Comp
+L power:VSS #PWR0105
+U 1 1 5B7AC5E5
+P 2000 2450
+F 0 "#PWR0105" H 2000 2300 50  0001 C CNN
+F 1 "VSS" V 2017 2578 50  0000 L CNN
+F 2 "" H 2000 2450 50  0001 C CNN
+F 3 "" H 2000 2450 50  0001 C CNN
+	1    2000 2450
+	0    1    1    0
+$EndComp
+$Comp
+L power:VSS #PWR0106
+U 1 1 5B7AC5F8
+P 1100 2450
+F 0 "#PWR0106" H 1100 2300 50  0001 C CNN
+F 1 "VSS" V 1118 2578 50  0000 L CNN
+F 2 "" H 1100 2450 50  0001 C CNN
+F 3 "" H 1100 2450 50  0001 C CNN
+	1    1100 2450
+	0    -1   -1   0
+$EndComp
+$Comp
+L power:VDDA #PWR0107
+U 1 1 5B7AC66D
+P 2000 2550
+F 0 "#PWR0107" H 2000 2400 50  0001 C CNN
+F 1 "VDDA" V 2017 2678 50  0000 L CNN
+F 2 "" H 2000 2550 50  0001 C CNN
+F 3 "" H 2000 2550 50  0001 C CNN
+	1    2000 2550
+	0    1    1    0
+$EndComp
+$Comp
+L power:VDDA #PWR0108
+U 1 1 5B7AC69F
+P 1100 2550
+F 0 "#PWR0108" H 1100 2400 50  0001 C CNN
+F 1 "VDDA" V 1118 2678 50  0000 L CNN
+F 2 "" H 1100 2550 50  0001 C CNN
+F 3 "" H 1100 2550 50  0001 C CNN
+	1    1100 2550
+	0    -1   -1   0
+$EndComp
+$Comp
+L power:VSSA #PWR0109
+U 1 1 5B7AC72D
+P 1100 2650
+F 0 "#PWR0109" H 1100 2500 50  0001 C CNN
+F 1 "VSSA" V 1118 2777 50  0000 L CNN
+F 2 "" H 1100 2650 50  0001 C CNN
+F 3 "" H 1100 2650 50  0001 C CNN
+	1    1100 2650
+	0    -1   -1   0
+$EndComp
+$Comp
+L power:VSSA #PWR0110
+U 1 1 5B7AC753
+P 2000 2650
+F 0 "#PWR0110" H 2000 2500 50  0001 C CNN
+F 1 "VSSA" V 2017 2778 50  0000 L CNN
+F 2 "" H 2000 2650 50  0001 C CNN
+F 3 "" H 2000 2650 50  0001 C CNN
+	1    2000 2650
+	0    1    1    0
+$EndComp
+$Comp
+L power:VCC #PWR0111
+U 1 1 5B7AC7C1
+P 2000 2350
+F 0 "#PWR0111" H 2000 2200 50  0001 C CNN
+F 1 "VCC" V 2017 2478 50  0000 L CNN
+F 2 "" H 2000 2350 50  0001 C CNN
+F 3 "" H 2000 2350 50  0001 C CNN
+	1    2000 2350
+	0    1    1    0
+$EndComp
+$Comp
+L power:VCC #PWR0112
+U 1 1 5B7AC7DF
+P 1100 2350
+F 0 "#PWR0112" H 1100 2200 50  0001 C CNN
+F 1 "VCC" V 1118 2477 50  0000 L CNN
+F 2 "" H 1100 2350 50  0001 C CNN
+F 3 "" H 1100 2350 50  0001 C CNN
+	1    1100 2350
+	0    -1   -1   0
+$EndComp
+Wire Wire Line
+	1100 2550 1150 2550
+Wire Wire Line
+	1150 2650 1100 2650
+Wire Wire Line
+	1100 2450 1150 2450
+Wire Wire Line
+	1150 2350 1100 2350
+Wire Wire Line
+	1950 2350 2000 2350
+Wire Wire Line
+	2000 2450 1950 2450
+Wire Wire Line
+	1950 2550 2000 2550
+Wire Wire Line
+	2000 2650 1950 2650
+$Comp
+L Mechanical:MountingHole MH2
+U 1 1 5B7AD009
+P 1300 7650
+F 0 "MH2" H 1400 7696 50  0000 L CNN
+F 1 "MountingHole" H 1400 7605 50  0000 L CNN
+F 2 "SquantorPcbOutline:MountingHole_2.5mm_no_metal" H 1300 7650 50  0001 C CNN
+F 3 "~" H 1300 7650 50  0001 C CNN
+	1    1300 7650
+	1    0    0    -1
+$EndComp
+$Comp
+L Mechanical:MountingHole MH1
+U 1 1 5B7AD05B
+P 1300 7400
+F 0 "MH1" H 1400 7446 50  0000 L CNN
+F 1 "MountingHole" H 1400 7355 50  0000 L CNN
+F 2 "SquantorPcbOutline:MountingHole_2.5mm_no_metal" H 1300 7400 50  0001 C CNN
+F 3 "~" H 1300 7400 50  0001 C CNN
+	1    1300 7400
 	1    0    0    -1
 $EndComp
