File: Hammond_1551G_OSH2L_devboard/Hammond_1551G_OSH2L_devboard.sch (KiCad schematic (older format))
At the start: 6 parts, among them J1 DevBoardDigital, J2 DevBoardAnalog

Commit message: updated devboard pinout
Connections:
- net labels added: +BATT, VBUS
- net labels removed: VCC
Changed lines of the file:
@@
 EESchema Schematic File Version 4
-LIBS:NiBeetle_JLCPCB_4layer-cache
+LIBS:Hammond_1551G_OSH2L_devboard-cache
 EELAYER 26 0
 EELAYER END
@@
 $EndComp
 $Comp
-L power:VSS #PWR0105
-U 1 1 5B7AC5E5
-P 2000 2450
-F 0 "#PWR0105" H 2000 2300 50  0001 C CNN
-F 1 "VSS" V 2017 2578 50  0000 L CNN
-F 2 "" H 2000 2450 50  0001 C CNN
-F 3 "" H 2000 2450 50  0001 C CNN
-	1    2000 2450
-	0    1    1    0
-$EndComp
-$Comp
-L power:VSS #PWR0106
-U 1 1 5B7AC5F8
-P 1100 2450
-F 0 "#PWR0106" H 1100 2300 50  0001 C CNN
-F 1 "VSS" V 1118 2578 50  0000 L CNN
-F 2 "" H 1100 2450 50  0001 C CNN
-F 3 "" H 1100 2450 50  0001 C CNN
-	1    1100 2450
-	0    -1   -1   0
-$EndComp
-$Comp
 L power:VDDA #PWR0107
 U 1 1 5B7AC66D
@@
 	0    1    1    0
 $EndComp
-$Comp
-L power:VCC #PWR0111
-U 1 1 5B7AC7C1
-P 2000 2350
-F 0 "#PWR0111" H 2000 2200 50  0001 C CNN
-F 1 "VCC" V 2017 2478 50  0000 L CNN
-F 2 "" H 2000 2350 50  0001 C CNN
-F 3 "" H 2000 2350 50  0001 C CNN
-	1    2000 2350
-	0    1    1    0
-$EndComp
-$Comp
-L power:VCC #PWR0112
-U 1 1 5B7AC7DF
-P 1100 2350
-F 0 "#PWR0112" H 1100 2200 50  0001 C CNN
-F 1 "VCC" V 1118 2477 50  0000 L CNN
-F 2 "" H 1100 2350 50  0001 C CNN
-F 3 "" H 1100 2350 50  0001 C CNN
-	1    1100 2350
-	0    -1   -1   0
-$EndComp
 Wire Wire Line
 	1100 2550 1150 2550
@@
 	1    0    0    -1
 $EndComp
+$Comp
+L power:+BATT #PWR?
+U 1 1 5C4A395A
+P 2000 2450
+F 0 "#PWR?" H 2000 2300 50  0001 C CNN
+F 1 "+BATT" V 2015 2578 50  0000 L CNN
+F 2 "" H 2000 2450 50  0001 C CNN
+F 3 "" H 2000 2450 50  0001 C CNN
+	1    2000 2450
+	0    1    1    0
+$EndComp
+$Comp
+L power:+BATT #PWR?
+U 1 1 5C4A3990
+P 1100 2450
+F 0 "#PWR?" H 1100 2300 50  0001 C CNN
+F 1 "+BATT" V 1115 2577 50  0000 L CNN
+F 2 "" H 1100 2450 50  0001 C CNN
+F 3 "" H 1100 2450 50  0001 C CNN
+	1    1100 2450
+	0    -1   -1   0
+$EndComp
+$Comp
+L power:VBUS #PWR?
+U 1 1 5C4A39D0
+P 2000 2350
+F 0 "#PWR?" H 2000 2200 50  0001 C CNN
+F 1 "VBUS" V 2015 2478 50  0000 L CNN
+F 2 "" H 2000 2350 50  0001 C CNN
+F 3 "" H 2000 2350 50  0001 C CNN
+	1    2000 2350
+	0    1    1    0
+$EndComp
+$Comp
+L power:VBUS #PWR?
+U 1 1 5C4A39F4
+P 1100 2350
+F 0 "#PWR?" H 1100 2200 50  0001 C CNN
+F 1 "VBUS" V 1115 2477 50  0000 L CNN
+F 2 "" H 1100 2350 50  0001 C CNN
+F 3 "" H 1100 2350 50  0001 C CNN
+	1    1100 2350
+	0    -1   -1   0
+$EndComp
 $EndSCHEMATC
