File: Hammond_1551M_OSH2layer/Hammond_1551M_OSH2layer.kicad_pcb (KiCad board)
At the start: 2 copper layers, 29 x 29 mm, 4 parts

Commit message: updated Hammond 1551M template
Parts:
- N2: value 20190307 -> 20190520
Other:
- outline, holes or cut-outs redrawn
Changed lines of the file:
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@@
-(kicad_pcb (version 20171130) (host pcbnew 5.0.2-bee76a0~70~ubuntu18.04.1)
+(kicad_pcb (version 20171130) (host pcbnew 5.1.2-f72e74a~84~ubuntu18.04.1)
   (general
     (thickness 1.6)
@@
     (zone_45_only no)
     (trace_min 0.1524)
-    (segment_width 0.2)
-    (edge_width 0.15)
     (via_size 0.381)
     (via_drill 0.254)
@@
     (uvia_min_size 0.381)
     (uvia_min_drill 0.254)
+    (edge_width 0.15)
+    (segment_width 0.2)
     (pcb_text_width 0.3)
     (pcb_text_size 1.5 1.5)
@@
       (effects (font (size 1 1) (thickness 0.15)))
     )
-    (fp_text value 20190307 (at -0.4 -0.1) (layer F.SilkS)
+    (fp_text value 20190520 (at -0.4 -0.1) (layer F.SilkS)
       (effects (font (size 1 1) (thickness 0.15)))
     )
@@
     (pad "" np_thru_hole circle (at 0 0) (size 2.5 2.5) (drill 2.5) (layers *.Cu *.Mask))
   )
-  (gr_arc (start 138.649999 110.55) (end 141.649999 110.55) (angle -89.9999809) (layer Edge.Cuts) (width 0.15))
-  (gr_arc (start 161.9 95.55) (end 162.4 95.55) (angle -90) (layer Edge.Cuts) (width 0.15))
+  (gr_arc (start 136.65 112.549583) (end 139.65 112.549583) (angle -90.95484125) (layer Edge.Cuts) (width 0.15))
+  (gr_arc (start 161.9 93.55) (end 162.4 93.55) (angle -90) (layer Edge.Cuts) (width 0.15))
   (gr_arc (start 161.9 115.3) (end 161.9 115.8) (angle -90) (layer Edge.Cuts) (width 0.15))
-  (gr_arc (start 142.15 115.3) (end 141.65 115.3) (angle -90) (layer Edge.Cuts) (width 0.15))
-  (gr_arc (start 133.9 107.05) (end 133.4 107.05) (angle -90) (layer Edge.Cuts) (width 0.15))
+  (gr_arc (start 140.15 115.3) (end 139.65 115.3) (angle -90) (layer Edge.Cuts) (width 0.15))
+  (gr_arc (start 133.9 109.05) (end 133.4 109.05) (angle -90) (layer Edge.Cuts) (width 0.15))
   (gr_arc (start 133.9 87.3) (end 133.9 86.8) (angle -90) (layer Edge.Cuts) (width 0.15))
-  (gr_line (start 133.4 107.05) (end 133.4 87.3) (layer Edge.Cuts) (width 0.15))
-  (gr_line (start 138.65 107.55) (end 133.9 107.55) (layer Edge.Cuts) (width 0.15))
-  (gr_line (start 141.65 115.3) (end 141.65 110.55) (layer Edge.Cuts) (width 0.15))
-  (gr_line (start 161.9 115.8) (end 142.15 115.8) (layer Edge.Cuts) (width 0.15))
-  (gr_line (start 162.4 95.55) (end 162.4 115.3) (layer Edge.Cuts) (width 0.15))
-  (gr_line (start 157.15 95.05) (end 161.9 95.05) (layer Edge.Cuts) (width 0.15))
-  (gr_arc (start 157.15 92.05) (end 154.15 92.05) (angle -89.9999809) (layer Edge.Cuts) (width 0.15))
-  (gr_line (start 154.15 87.3) (end 154.15 92.05) (layer Edge.Cuts) (width 0.15))
-  (gr_arc (start 153.65 87.3) (end 154.15 87.3) (angle -90) (layer Edge.Cuts) (width 0.15))
-  (gr_line (start 133.9 86.8) (end 153.65 86.8) (layer Edge.Cuts) (width 0.15))
+  (gr_line (start 133.4 109.05) (end 133.4 87.3) (layer Edge.Cuts) (width 0.15))
+  (gr_line (start 136.600007 109.55) (end 133.9 109.55) (layer Edge.Cuts) (width 0.15))
+  (gr_line (start 139.65 115.3) (end 139.65 112.549583) (layer Edge.Cuts) (width 0.15))
+  (gr_line (start 161.9 115.8) (end 140.15 115.8) (layer Edge.Cuts) (width 0.15))
+  (gr_line (start 162.4 93.55) (end 162.4 115.3) (layer Edge.Cuts) (width 0.15))
+  (gr_line (start 159.149999 93.05) (end 161.9 93.05) (layer Edge.Cuts) (width 0.15))
+  (gr_arc (start 159.15 90.05) (end 156.15 90.05) (angle -89.9999809) (layer Edge.Cuts) (width 0.15))
+  (gr_line (start 156.15 87.3) (end 156.15 90.05) (layer Edge.Cuts) (width 0.15))
+  (gr_arc (start 155.65 87.3) (end 156.15 87.3) (angle -90) (layer Edge.Cuts) (width 0.15))
+  (gr_line (start 133.9 86.8) (end 155.65 86.8) (layer Edge.Cuts) (width 0.15))
 )
