File: small_nuclone_devboard_2_layer/microcontroller.kicad_sch (KiCad schematic)
At the start: 2 parts, among them J5 Conn_02x06_Odd_Even

Commit message: updates
Other:
- moved on the sheet: J5
Changed lines of the file:
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@@
 (kicad_sch (version 20230121) (generator eeschema)
   (paper "A4")
-  (junction (at 146.05 171.45) (diameter 0) (color 0 0 0 0)
-  )
-  (junction (at 146.05 173.99) (diameter 0) (color 0 0 0 0)
-  )
-  (junction (at 146.05 176.53) (diameter 0) (color 0 0 0 0)
+  (junction (at 146.05 179.07) (diameter 0) (color 0 0 0 0)
+  )
+  (junction (at 146.05 181.61) (diameter 0) (color 0 0 0 0)
+  )
+  (junction (at 146.05 184.15) (diameter 0) (color 0 0 0 0)
   )
   (junction (at 25.4 33.02) (diameter 0) (color 0 0 0 0)
@@
     (stroke (width 0) (type default))
   )
-  (wire (pts (xy 146.05 171.45) (xy 147.32 171.45))
-    (stroke (width 0) (type default))
-  )
-  (polyline (pts (xy 175.26 186.69) (xy 175.26 187.96))
-    (stroke (width 0) (type default))
-  )
-  (wire (pts (xy 160.02 171.45) (xy 161.29 171.45))
-    (stroke (width 0) (type default))
-  )
-  (polyline (pts (xy 139.7 187.96) (xy 175.26 187.96))
+  (wire (pts (xy 146.05 179.07) (xy 147.32 179.07))
+    (stroke (width 0) (type default))
+  )
+  (polyline (pts (xy 175.26 194.31) (xy 175.26 195.58))
+    (stroke (width 0) (type default))
+  )
+  (wire (pts (xy 160.02 179.07) (xy 161.29 179.07))
+    (stroke (width 0) (type default))
+  )
+  (polyline (pts (xy 139.7 195.58) (xy 175.26 195.58))
     (stroke (width 0) (type default))
   )
@@
     (stroke (width 0) (type default))
   )
-  (wire (pts (xy 146.05 176.53) (xy 146.05 179.07))
-    (stroke (width 0) (type default))
-  )
-  (polyline (pts (xy 175.26 166.37) (xy 139.7 166.37))
+  (wire (pts (xy 146.05 184.15) (xy 146.05 186.69))
+    (stroke (width 0) (type default))
+  )
+  (polyline (pts (xy 175.26 173.99) (xy 139.7 173.99))
     (stroke (width 0) (type default))
   )
@@
     (stroke (width 0) (type default))
   )
-  (polyline (pts (xy 139.7 166.37) (xy 139.7 187.96))
-    (stroke (width 0) (type default))
-  )
-  (wire (pts (xy 160.02 179.07) (xy 161.29 179.07))
-    (stroke (width 0) (type default))
-  )
-  (wire (pts (xy 146.05 173.99) (xy 146.05 176.53))
-    (stroke (width 0) (type default))
-  )
-  (polyline (pts (xy 175.26 184.15) (xy 165.1 184.15))
+  (polyline (pts (xy 139.7 173.99) (xy 139.7 195.58))
+    (stroke (width 0) (type default))
+  )
+  (wire (pts (xy 160.02 186.69) (xy 161.29 186.69))
+    (stroke (width 0) (type default))
+  )
+  (wire (pts (xy 146.05 181.61) (xy 146.05 184.15))
+    (stroke (width 0) (type default))
+  )
+  (polyline (pts (xy 175.26 191.77) (xy 165.1 191.77))
     (stroke (width 0) (type default))
   )
@@
     (stroke (width 0) (type default))
   )
-  (wire (pts (xy 160.02 176.53) (xy 161.29 176.53))
-    (stroke (width 0) (type default))
-  )
-  (polyline (pts (xy 175.26 186.69) (xy 175.26 166.37))
+  (wire (pts (xy 160.02 184.15) (xy 161.29 184.15))
+    (stroke (width 0) (type default))
+  )
+  (polyline (pts (xy 175.26 194.31) (xy 175.26 173.99))
     (stroke (width 0) (type default))
   )
@@
     (stroke (width 0) (type default))
   )
-  (wire (pts (xy 144.78 171.45) (xy 146.05 171.45))
-    (stroke (width 0) (type default))
-  )
-  (wire (pts (xy 160.02 173.99) (xy 161.29 173.99))
+  (wire (pts (xy 144.78 179.07) (xy 146.05 179.07))
+    (stroke (width 0) (type default))
+  )
+  (wire (pts (xy 160.02 181.61) (xy 161.29 181.61))
     (stroke (width 0) (type default))
   )
@@
     (stroke (width 0) (type default))
   )
-  (wire (pts (xy 146.05 173.99) (xy 147.32 173.99))
-    (stroke (width 0) (type default))
-  )
-  (wire (pts (xy 146.05 176.53) (xy 147.32 176.53))
-    (stroke (width 0) (type default))
-  )
-  (wire (pts (xy 146.05 171.45) (xy 146.05 173.99))
+  (wire (pts (xy 146.05 181.61) (xy 147.32 181.61))
+    (stroke (width 0) (type default))
+  )
+  (wire (pts (xy 146.05 184.15) (xy 147.32 184.15))
+    (stroke (width 0) (type default))
+  )
+  (wire (pts (xy 146.05 179.07) (xy 146.05 181.61))
     (stroke (width 0) (type default))
   )
@@
     (stroke (width 0) (type default))
   )
-  (polyline (pts (xy 165.1 184.15) (xy 165.1 187.96))
-    (stroke (width 0) (type default))
-  )
-  (wire (pts (xy 146.05 179.07) (xy 147.32 179.07))
-    (stroke (width 0) (type default))
-  )
-  (text "Testpads" (at 166.37 186.69 0)
+  (polyline (pts (xy 165.1 191.77) (xy 165.1 195.58))
+    (stroke (width 0) (type default))
+  )
+  (wire (pts (xy 146.05 186.69) (xy 147.32 186.69))
+    (stroke (width 0) (type default))
+  )
+  (text "Testpads" (at 166.37 194.31 0)
     (effects (font (size 1.27 1.27)) (justify left bottom))
   )
@@
     (effects (font (size 1.27 1.27)) (justify left bottom))
   )
-  (label "BOOTLOADER" (at 161.29 179.07 0) (fields_autoplaced)
-    (effects (font (size 1.27 1.27)) (justify left bottom))
-  )
-  (label "TCK" (at 161.29 173.99 0) (fields_autoplaced)
+  (label "BOOTLOADER" (at 161.29 186.69 0) (fields_autoplaced)
+    (effects (font (size 1.27 1.27)) (justify left bottom))
+  )
+  (label "TCK" (at 161.29 181.61 0) (fields_autoplaced)
     (effects (font (size 1.27 1.27)) (justify left bottom))
   )
@@
     (effects (font (size 1.27 1.27)) (justify left bottom))
   )
-  (label "TMS" (at 161.29 176.53 0) (fields_autoplaced)
-    (effects (font (size 1.27 1.27)) (justify left bottom))
-  )
-  (label "VSS" (at 144.78 171.45 180) (fields_autoplaced)
+  (label "TMS" (at 161.29 184.15 0) (fields_autoplaced)
+    (effects (font (size 1.27 1.27)) (justify left bottom))
+  )
+  (label "VSS" (at 144.78 179.07 180) (fields_autoplaced)
     (effects (font (size 1.27 1.27)) (justify right bottom))
   )
@@
     (effects (font (size 1.27 1.27)) (justify left bottom))
   )
-  (label "RESET" (at 161.29 171.45 0) (fields_autoplaced)
+  (label "RESET" (at 161.29 179.07 0) (fields_autoplaced)
     (effects (font (size 1.27 1.27)) (justify left bottom))
   )
@@
     )
   )
-  (symbol (lib_id "Connector_Generic:Conn_02x04_Odd_Even") (at 152.4 173.99 0) (unit 1)
+  (symbol (lib_id "Connector_Generic:Conn_02x04_Odd_Even") (at 152.4 181.61 0) (unit 1)
     (in_bom yes) (on_board yes) (dnp no)
-    (property "Reference" "J5" (at 152.4 168.91 0)
+    (property "Reference" "J5" (at 152.4 176.53 0)
       (effects (font (size 1.27 1.27)))
     )
-    (property "Value" "Conn_02x06_Odd_Even" (at 153.67 181.61 0)
+    (property "Value" "Conn_02x06_Odd_Even" (at 153.67 189.23 0)
       (effects (font (size 1.27 1.27)))
     )
-    (property "Footprint" "SquantorConnectors:Header-0127-2X04-H006" (at 152.4 173.99 0)
+    (property "Footprint" "SquantorConnectors:Header-0127-2X04-H006" (at 152.4 181.61 0)
       (effects (font (size 1.27 1.27)) hide)
     )
-    (property "Datasheet" "~" (at 152.4 173.99 0)
+    (property "Datasheet" "~" (at 152.4 181.61 0)
       (effects (font (size 1.27 1.27)) hide)
     )
