File: nuclone_devboard_small_2_layer/microcontroller.kicad_sch (KiCad schematic)
At the start: 2 parts, among them J5 Conn_02x06_Odd_Even

Commit message: WIP redoing the template
Parts:
- C3: footprint SquantorRcl:C_0603 -> SquantorCapacitor:C_0603
Changed lines of the file:
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@@
     (effects (font (size 1.27 1.27)) (justify left bottom))
   )
-  (label "BOOTLOADER" (at 25.4 50.8 0) (fields_autoplaced)
+  (label "BOOT" (at 25.4 50.8 0) (fields_autoplaced)
     (effects (font (size 1.27 1.27)) (justify left bottom))
   )
@@
     (effects (font (size 1.27 1.27)) (justify left bottom))
   )
-  (label "BOOTLOADER" (at 161.29 186.69 0) (fields_autoplaced)
+  (label "BOOT" (at 161.29 186.69 0) (fields_autoplaced)
     (effects (font (size 1.27 1.27)) (justify left bottom))
   )
@@
       (effects (font (size 1.27 1.27)) (justify left))
     )
-    (property "Footprint" "SquantorRcl:C_0603" (at 26.3652 31.75 0)
+    (property "Footprint" "SquantorCapacitor:C_0603" (at 26.3652 31.75 0)
       (effects (font (size 1.27 1.27)) hide)
     )
@@
     (pin "2")
     (instances
-      (project "small_nuclone_devboard_2_layer"
+      (project "nuclone_devboard_small_2_layer"
         (path "/937928d4-4dfb-4f2f-91d0-697ec54ac283/00000000-0000-0000-0000-00006127a958"
           (reference "C3") (unit 1)
@@
     (pin "8")
     (instances
-      (project "small_nuclone_devboard_2_layer"
+      (project "nuclone_devboard_small_2_layer"
         (path "/937928d4-4dfb-4f2f-91d0-697ec54ac283/00000000-0000-0000-0000-00006127a958"
           (reference "J5") (unit 1)
